File: kicad/password.sch (KiCad schematic (older format))
At the start: 54 parts, among them CON1 AVR-ISP-6, CON2 USB-MICRO-B2, P1 CONN_4, Q1 MOS_P, Q2 MOS_N, Q3 MOS_P, SW1 SW_PUSH, U1 CON_FPC_30, U2 CON_SMARTC, U3 IP4234CZ6,125, U4 ATMEGA32U4_QFN, U5 ST662ACD, U6 AT45DB011D, X1 16MHz

Commit message: adding the PCB
Parts:
- R7: value 3k3 -> 4k7
Changed lines of the file:
@@
 Sheet 1 1
 Title ""
-Date "18 dec 2013"
+Date "4 jan 2014"
 Rev ""
 Comp ""
@@
 P 9500 2050
 F 0 "R7" V 9580 2050 40  0000 C CNN
-F 1 "3k3" V 9507 2051 40  0000 C CNN
+F 1 "4k7" V 9507 2051 40  0000 C CNN
 F 2 "~" V 9430 2050 30  0000 C CNN
 F 3 "~" H 9500 2050 30  0000 C CNN
@@
 P 3650 3750
 F 0 "R7" V 3730 3750 40  0000 C CNN
-F 1 "3k3" V 3657 3751 40  0000 C CNN
+F 1 "4k7" V 3657 3751 40  0000 C CNN
 F 2 "~" V 3580 3750 30  0000 C CNN
 F 3 "~" H 3650 3750 30  0000 C CNN
@@
 P 5550 6925
 F 0 "R7" V 5630 6925 40  0000 C CNN
-F 1 "3k3" V 5557 6926 40  0000 C CNN
+F 1 "4k7" V 5557 6926 40  0000 C CNN
 F 2 "~" V 5480 6925 30  0000 C CNN
 F 3 "~" H 5550 6925 30  0000 C CNN
@@
 P 5850 6925
 F 0 "R7" V 5930 6925 40  0000 C CNN
-F 1 "3k3" V 5857 6926 40  0000 C CNN
+F 1 "4k7" V 5857 6926 40  0000 C CNN
 F 2 "~" V 5780 6925 30  0000 C CNN
 F 3 "~" H 5850 6925 30  0000 C CNN
@@
 P 5700 6925
 F 0 "R7" V 5780 6925 40  0000 C CNN
-F 1 "3k3" V 5707 6926 40  0000 C CNN
+F 1 "4k7" V 5707 6926 40  0000 C CNN
 F 2 "~" V 5630 6925 30  0000 C CNN
 F 3 "~" H 5700 6925 30  0000 C CNN
@@
 P 6000 6925
 F 0 "R7" V 6080 6925 40  0000 C CNN
-F 1 "3k3" V 6007 6926 40  0000 C CNN
+F 1 "4k7" V 6007 6926 40  0000 C CNN
 F 2 "~" V 5930 6925 30  0000 C CNN
 F 3 "~" H 6000 6925 30  0000 C CNN
@@
 P 5400 6925
 F 0 "R7" V 5480 6925 40  0000 C CNN
-F 1 "3k3" V 5407 6926 40  0000 C CNN
+F 1 "4k7" V 5407 6926 40  0000 C CNN
 F 2 "~" V 5330 6925 30  0000 C CNN
 F 3 "~" H 5400 6925 30  0000 C CNN
@@
 P 6150 6925
 F 0 "R7" V 6230 6925 40  0000 C CNN
-F 1 "3k3" V 6157 6926 40  0000 C CNN
+F 1 "4k7" V 6157 6926 40  0000 C CNN
 F 2 "~" V 6080 6925 30  0000 C CNN
 F 3 "~" H 6150 6925 30  0000 C CNN

Commit message: update schematics
Parts:
- added C3: 10uF, ~, symbol C
- C18: value 100nF -> 4.7uF
- C20: value 4.7uF -> 100nF
- C9: value 4.7uF / 25V -> 10uF
Connections:
- net 12V_FILT: now also C3.1
- net GND: now also C3.2
Other:
- note removed: "(tantal)"
- moved on the sheet: C1, C2, C4, C5
Changed lines of the file:
@@
 Sheet 1 1
 Title ""
-Date "4 jan 2014"
+Date "6 jan 2014"
 Rev ""
 Comp ""
@@
 P 3000 4950
 F 0 "C9" H 3000 5050 40  0000 L CNN
-F 1 "4.7uF / 25V" H 3006 4865 40  0000 L CNN
+F 1 "10uF" H 3006 4865 40  0000 L CNN
 F 2 "~" H 3038 4800 30  0000 C CNN
 F 3 "~" H 3000 4950 60  0000 C CNN
@@
 L C C1
 U 1 1 5289A0B1
-P 950 5350
-F 0 "C1" H 950 5450 40  0000 L CNN
-F 1 "10uF" H 956 5265 40  0000 L CNN
-F 2 "~" H 988 5200 30  0000 C CNN
-F 3 "~" H 950 5350 60  0000 C CNN
-	1    950  5350
+P 800 5350
+F 0 "C1" H 800 5450 40  0000 L CNN
+F 1 "10uF" H 806 5265 40  0000 L CNN
+F 2 "~" H 838 5200 30  0000 C CNN
+F 3 "~" H 800 5350 60  0000 C CNN
+	1    800  5350
 	1    0    0    -1
 $EndComp
@@
 L C C4
 U 1 1 5289A0BC
-P 1200 5350
-F 0 "C4" H 1200 5450 40  0000 L CNN
-F 1 "100nF" H 1206 5265 40  0000 L CNN
-F 2 "~" H 1238 5200 30  0000 C CNN
-F 3 "~" H 1200 5350 60  0000 C CNN
-	1    1200 5350
+P 1300 5350
+F 0 "C4" H 1300 5450 40  0000 L CNN
+F 1 "100nF" H 1306 5265 40  0000 L CNN
+F 2 "~" H 1338 5200 30  0000 C CNN
+F 3 "~" H 1300 5350 60  0000 C CNN
+	1    1300 5350
 	1    0    0    -1
 $EndComp
@@
 L GND #PWR036
 U 1 1 5289A0C2
-P 950 5650
-F 0 "#PWR036" H 950 5650 30  0001 C CNN
-F 1 "GND" H 950 5580 30  0001 C CNN
-F 2 "" H 950 5650 60  0000 C CNN
-F 3 "" H 950 5650 60  0000 C CNN
-	1    950  5650
+P 1050 5650
+F 0 "#PWR036" H 1050 5650 30  0001 C CNN
+F 1 "GND" H 1050 5580 30  0001 C CNN
+F 2 "" H 1050 5650 60  0000 C CNN
+F 3 "" H 1050 5650 60  0000 C CNN
+	1    1050 5650
 	1    0    0    -1
 $EndComp
@@
 L +3.3V #PWR039
 U 1 1 5289B36B
-P 950 5950
-F 0 "#PWR039" H 950 5910 30  0001 C CNN
-F 1 "+3.3V" H 950 6060 30  0000 C CNN
-F 2 "" H 950 5950 60  0000 C CNN
-F 3 "" H 950 5950 60  0000 C CNN
-	1    950  5950
+P 1050 5950
+F 0 "#PWR039" H 1050 5910 30  0001 C CNN
+F 1 "+3.3V" H 1050 6060 30  0000 C CNN
+F 2 "" H 1050 5950 60  0000 C CNN
+F 3 "" H 1050 5950 60  0000 C CNN
+	1    1050 5950
 	1    0    0    -1
 $EndComp
@@
 L C C2
 U 1 1 5289B371
-P 950 6250
-F 0 "C2" H 950 6350 40  0000 L CNN
-F 1 "4.7uF" H 956 6165 40  0000 L CNN
-F 2 "~" H 988 6100 30  0000 C CNN
-F 3 "~" H 950 6250 60  0000 C CNN
-	1    950  6250
+P 1050 6250
+F 0 "C2" H 1050 6350 40  0000 L CNN
+F 1 "4.7uF" H 1056 6165 40  0000 L CNN
+F 2 "~" H 1088 6100 30  0000 C CNN
+F 3 "~" H 1050 6250 60  0000 C CNN
+	1    1050 6250
 	1    0    0    -1
 $EndComp
@@
 L C C5
 U 1 1 5289B37C
-P 1200 6250
-F 0 "C5" H 1200 6350 40  0000 L CNN
-F 1 "100nF" H 1206 6165 40  0000 L CNN
-F 2 "~" H 1238 6100 30  0000 C CNN
-F 3 "~" H 1200 6250 60  0000 C CNN
-	1    1200 6250
+P 1300 6250
+F 0 "C5" H 1300 6350 40  0000 L CNN
+F 1 "100nF" H 1306 6165 40  0000 L CNN
+F 2 "~" H 1338 6100 30  0000 C CNN
+F 3 "~" H 1300 6250 60  0000 C CNN
+	1    1300 6250
 	1    0    0    -1
 $EndComp
@@
 L GND #PWR040
 U 1 1 5289B382
-P 950 6550
-F 0 "#PWR040" H 950 6550 30  0001 C CNN
-F 1 "GND" H 950 6480 30  0001 C CNN
-F 2 "" H 950 6550 60  0000 C CNN
-F 3 "" H 950 6550 60  0000 C CNN
-	1    950  6550
-	1    0    0    -1
-$EndComp
-Text Notes 3100 5150 0    60   ~ 0
-(tantal)
+P 1050 6550
+F 0 "#PWR040" H 1050 6550 30  0001 C CNN
+F 1 "GND" H 1050 6480 30  0001 C CNN
+F 2 "" H 1050 6550 60  0000 C CNN
+F 3 "" H 1050 6550 60  0000 C CNN
+	1    1050 6550
+	1    0    0    -1
+$EndComp
 $Comp
 L C C10
@@
 P 8300 6550
 F 0 "C20" H 8300 6650 40  0000 L CNN
-F 1 "4.7uF" H 8306 6465 40  0000 L CNN
+F 1 "100nF" H 8306 6465 40  0000 L CNN
 F 2 "~" H 8338 6400 30  0000 C CNN
 F 3 "~" H 8300 6550 60  0000 C CNN
@@
 P 7250 6550
 F 0 "C18" H 7250 6650 40  0000 L CNN
-F 1 "100nF" H 7256 6465 40  0000 L CNN
+F 1 "4.7uF" H 7256 6465 40  0000 L CNN
 F 2 "~" H 7288 6400 30  0000 C CNN
 F 3 "~" H 7250 6550 60  0000 C CNN
@@
 Text Label 2650 4850 3    60   ~ 0
 12V_FILT
-Text Label 700  5100 0    60   ~ 0
+Text Label 850  5100 0    60   ~ 0
 12V_FILT
 $Comp
@@
 Wire Wire Line
 	3400 2700 3400 2600
-Connection ~ 950  5100
-Wire Wire Line
-	950  5150 950  5100
-Wire Wire Line
-	1200 5100 1200 5150
-Wire Wire Line
-	700  5100 1200 5100
+Connection ~ 1050 5100
+Wire Wire Line
+	1050 5150 1050 5100
+Wire Wire Line
+	1300 5100 1300 5150
+Wire Wire Line
+	800  5100 1300 5100
 Wire Wire Line
 	2650 4350 2650 7150
@@
 Wire Wire Line
 	2900 6750 2450 6750
-Connection ~ 950  6000
-Wire Wire Line
-	1200 6000 1200 6050
-Wire Wire Line
-	950  6000 1200 6000
-Wire Wire Line
-	950  5950 950  6050
-Connection ~ 950  6500
-Wire Wire Line
-	1200 6500 1200 6450
-Wire Wire Line
-	950  6500 1200 6500
-Wire Wire Line
-	950  6450 950  6550
+Connection ~ 1050 6000
+Wire Wire Line
+	1300 6000 1300 6050
+Wire Wire Line
+	1050 6000 1300 6000
+Wire Wire Line
+	1050 5950 1050 6050
+Connection ~ 1050 6500
+Wire Wire Line
+	1300 6500 1300 6450
+Wire Wire Line
+	1050 6500 1300 6500
+Wire Wire Line
+	1050 6450 1050 6550
 Connection ~ 2800 6650
 Wire Wire Line
@@
 Wire Wire Line
 	2650 7150 2450 7150
-Connection ~ 950  5600
-Wire Wire Line
-	1200 5600 1200 5550
-Wire Wire Line
-	950  5600 1200 5600
-Wire Wire Line
-	950  5550 950  5650
+Connection ~ 1050 5600
+Wire Wire Line
+	1300 5600 1300 5550
+Wire Wire Line
+	800  5600 1300 5600
+Wire Wire Line
+	1050 5550 1050 5650
 Wire Wire Line
 	2450 4550 2650 4550
@@
 Wire Notes Line
 	7475 1550 11225 1550
+$Comp
+L C C3
+U 1 1 52CB305A
+P 1050 5350
+F 0 "C3" H 1050 5450 40  0000 L CNN
+F 1 "10uF" H 1056 5265 40  0000 L CNN
+F 2 "~" H 1088 5200 30  0000 C CNN
+F 3 "~" H 1050 5350 60  0000 C CNN
+	1    1050 5350
+	1    0    0    -1
+$EndComp
+Wire Wire Line
+	800  5600 800  5550
+Wire Wire Line
+	800  5150 800  5100
 $EndSCHEMATC
