File: kicad/olivier_design_v1/mooltipass.sch (KiCad schematic (older format))
At the start: 55 parts, among them CON1 AVR-ISP-6, CON2 USB-MICRO-B2, P1 CONN_4, Q1 MOS_P, Q2 MOS_N, Q3 MOS_P, SW1 SW_PUSH, U1 CON_FPC_30, U2 CON_SMARTC, U3 IP4234CZ6,125, U4 ATMEGA32U4_QFN, U5 ST662ACD, U6 AT45DB011D, X1 16MHz

Commit message: adding olivier's design
Parts:
- removed P1: CONN_4, symbol CONN_4
- removed SW1: SW_PUSH, ~, symbol SW_PUSH
- removed U2: CON_SMARTC, symbol CON_SMARTCARD
- added P1, P4: CONN_8, symbol CONN_8
- added P2: CONN_6, symbol CONN_6
- added P3: CONN_10, symbol CONN_10
- added Q4: MOS_N, ~, symbol MOS_N
- added U2: CON_7312P0225A13LF, ~, symbol CON_SMARTCARD2
- added U7: CON_STACK_9, symbol CON_STACK_9
- CON2: value USB-MICRO-B2 -> CON_10118194-0001LF
- U1: value CON_FPC_30 -> CON_SFV30R-2STE1HLF
- U6: value AT45DB011D -> AT45DB011D-SSH
Connections:
- net labels added: AREF, I2C_SCL, I2C_SDA, LED_CAT, LED_PWM, PB1, PB2, PB3, PB4, PB5, PB6, PB7, PC6, PC7, PD0, PD1, PD2, PD3, PD4, PD5, PD6, PD7, PE2, PE6, PF0, PF1, PF4, PF5, PF6, PF7, nCHANGE
- net labels removed: 12V_FILT, ADC0, ADC1, ADC2, ADC3, nHWB
- wire segments 289 -> 336
- no-connect marks 10 -> 8
Other:
- note added: "12V GENERATION"
- note added: "3.3V"
- note added: "5V"
- note added: "ARDUINO HEADERS"
- note added: "AREF"
- note added: "FLASH MEMORY"
- note added: "GND"
- note added: "ISP"
- note added: "LED PWM"
- note added: "NC"
- note added: "OLED"
- note added: "PB4"
- note added: "PB5"
- note added: "PB6"
- note added: "PB7"
- note added: "PC6"
- note added: "PC7"
- note added: "PD0"
- note added: "PD0 (SCL)"
- note added: "PD1"
- note added: "PD1 (SDA)"
- note added: "PD2"
- note added: "PD3"
- note added: "PD4"
- note added: "PD6"
- note added: "PD7"
- note added: "PE6"
- note added: "PF0"
- note added: "PF1"
- note added: "PF4"
- note added: "PF5"
- note added: "PF6"
- note added: "PF7"
- note added: "PLANNED HEADERS:\n-"
- note added: "RESET"
- note added: "SMART CARD"
- note added: "SMART CARD POWER"
- note added: "STACKING HEADER"
- note added: "USB"
- note added: "VIN"
- note removed: "1"
- note removed: "M. Stephan - Offline Password Keeper Schematics (Licensed under CERN OHL V1.2)"
- moved on the sheet: C1, C10, C11, C12, C13, C14, C15, C16, C17, C18, C19, C2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
