File: kicad/olivier_design_v1/mooltipass.sch (KiCad schematic (older format))
At the start: 60 parts, among them CON1 AVR-ISP-6, CON2 CON_10118194-0001LF, P1 CONN_8, P2 CONN_6, P3 CONN_10, P4 CONN_8, Q1 MOS_P, Q2 MOS_N, Q3 MOS_P, Q4 MOS_N, U1 CON_SFV30R-2STE1HLF, U2 CON_7312P0225A13LF, U3 IP4234CZ6,125_ALT, U4 ATMEGA32U4_QFN, U5 ST662ACD, U6 AT45DB011D-SSH, U7 CON_STACK_9, X1 16MHz

Commit message: update schematics olivier
Parts:
- removed CON1: AVR-ISP-6, AVR-ISP-6, symbol AVR-ISP-6
- added P5, P6, P7, P8: CONN_1, symbol CONN_1
Connections:
- wire segments 339 -> 335
Other:
- note added: "FIX"
- note removed: "ISP"

Commit message: Adding presentation & schematics for Olivier's design
Parts:
- removed U3: IP4234CZ6,125_ALT, ~, symbol IP4234CZ6,125_ALT
- added R12: 2k2, ~, symbol R
- added U3: IP4234CZ6,125, ~, symbol IP4234CZ6,125
- R11: value 10k -> 2k2
Connections:
- net labels removed: PB1, PB2, PB3, PB7, PC7, PD0, PD1, PD5, PD6, PE2, PF4, PF5
- wire segments 335 -> 336
- no-connect marks 8 -> 10
Other:
- note added: "- A2 removed (PF5)\n- A3 removed (PF4)\n- D13 switched to SCK\n- D12 switched to MISO\n- D11 switched to MOSI"
- note added: "0"
- note added: "1"
- note added: "10"
- note added: "11"
- note added: "12"
- note added: "13"
- note added: "2"
- note added: "3"
- note added: "4"
- note added: "5"
- note added: "5V->3.3V SIGNAL CONVERSION"
- note added: "6"
- note added: "7"
- note added: "8"
- note added: "9"
- note added: "A0"
- note added: "A1"
- note added: "A2"
- note added: "A3"
- note added: "A4"
- note added: "A5"
- note added: "Differences with official \n Leonardo pinout:\n"
- note added: "MAIN MICROCONTROLLER"
- note added: "OLED SCREEN"
- note added: "SCL"
- note added: "SDA"
- note added: "Supported shields:\n- Seeed BT (D0 -> D7)\n- Ada PN532 (SCL/SDA)\n- Ada PN532 (4 Dx pins)\n\nNot supported:\n- Bluefruit EZ (D0 & D1)\n- Wifly shield\n\nto check:\n- Seeed NFC v2\n- Arduino WIFI\n- Ada CC3000"
- note removed: "OLED"
- note removed: "PB4"
- note removed: "PB5"
- note removed: "PB6"
- note removed: "PB7"
- note removed: "PC6"
- note removed: "PC7"
- note removed: "PD0"
- note removed: "PD0 (SCL)"
- note removed: "PD1"
- note removed: "PD1 (SDA)"
- note removed: "PD2"
- note removed: "PD3"
- note removed: "PD4"
- note removed: "PD6"
- note removed: "PD7"
- note removed: "PE6"
- note removed: "PF0"
- note removed: "PF1"
- note removed: "PF4"
- note removed: "PF5"
- note removed: "PF6"
- note removed: "PF7"
- note removed: "PLANNED HEADERS:\n-"
- moved on the sheet: C13, C14, C15, C16, C17, C19, C21, C24, C26, C29, P3, P4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
