File: kicad/olivier_design_v1/mooltipass.sch (KiCad schematic (older format))
At the start: 64 parts, among them CON2 CON_10118194-0001LF, P1 CONN_8, P2 CONN_6, P3 CONN_10, P4 CONN_8, P5 CONN_1, P6 CONN_1, P7 CONN_1, P8 CONN_1, Q1 MOS_P, Q2 MOS_N, Q3 MOS_P, Q4 MOS_N, U1 CON_SFV30R-2STE1HLF, U2 CON_7312P0225A13LF, U3 IP4234CZ6,125, U4 ATMEGA32U4_QFN, U5 ST662ACD, U6 AT45DB011D-SSH, U7 CON_STACK_9, X1 16MHz

Commit message: update schematics
Other:
- note added: "- LED:\n- SMC: 5mA\n- MCU: 15mA\n- OLED: 130mA\n- TOUCH: 1mA\n- FLASH: 20mA\n- RES NET: 7mA\n\nTOTAL: 178mA"
- note added: "Max. power consumptions"
Changed lines of the file:
@@
 Sheet 1 1
 Title "M. Stephan - Offline Password Keeper Schematics (Licensed under CERN OHL V1.2)"
-Date "23 feb 2014"
+Date "12 apr 2014"
 Rev "2"
 Comp ""
@@
 	4450 5000 3650 5000
 Wire Notes Line
-	4900 8300 4900 4450
+	4900 11100 4900 4450
 Wire Wire Line
 	2700 4850 2700 5000
@@
 5V->3.3V SIGNAL CONVERSION
 Wire Notes Line
-	650  11100 3450 11100
+	650  11100 4900 11100
 Text Notes 9400 4750 0    60   ~ 0
 MAIN MICROCONTROLLER
@@
 	8050 5550 8050 5600
 Connection ~ 8050 5600
+Text Notes 3600 8450 0    60   ~ 0
+Max. power consumptions
+Text Notes 3600 8750 0    60   ~ 0
+- LED:\n- SMC: 5mA\n- MCU: 15mA\n- OLED: 130mA\n- TOUCH: 1mA\n- FLASH: 20mA\n- RES NET: 7mA\n\nTOTAL: 178mA
 $EndSCHEMATC

Commit message: final PCBs!
Parts:
- added F1: FUSE, ~, symbol FUSE
Connections:
- net VCC: now reaches C7.1, FB1.1, U3.5 (VCC)
- net VCC: now also F1.2; no longer CON2.1 (VBUS)
- new net: CON2.1 (VBUS), F1.1
Other:
- note added: "- LED: 30mA\n- SMC: 5mA\n- MCU: 15mA\n- OLED: 130mA\n- TOUCH: 1mA\n- FLASH: 20mA\n- RES NET: 7mA\n\nTOTAL: 208mA"
- note added: "Copyright Mathieu Stephan, 2014\n\nThis documentation describes Open Hardware and is licensed under the\nCERN OHL v. 1.2.\n\nYou may redistribute and modify this documentation under the terms of the\nCERN OHL v.1.2. (http://ohwr.org/cernohl). This documentation is distributed\nWITHOUT ANY EXPRESS OR IMPLIED WARRANTY, INCLUDING OF MERCHANTABILITY,\nSATISFACTORY QUALITY AND FITNESS FOR A PARTICULAR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"
- note removed: "- LED:\n- SMC: 5mA\n- MCU: 15mA\n- OLED: 130mA\n- TOUCH: 1mA\n- FLASH: 20mA\n- RES NET: 7mA\n\nTOTAL: 178mA"
- note removed: "Copyright Mathieu Stephan, 2013\n\nThis documentation describes Open Hardware and is licensed under the\nCERN OHL v. 1.2.\n\nYou may redistribute and modify this documentation under the terms of the\nCERN OHL v.1.2. (http://ohwr.org/cernohl). This documentation is distributed\nWITHOUT ANY EXPRESS OR IMPLIED WARRANTY, INCLUDING OF MERCHANTABILITY,\nSATISFACTORY QUALITY AND FITNESS FOR A PARTICULAR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"
- moved on the sheet: C7, CON2

Commit message: bom & schematics update
Parts:
- C1, C3: value 10uF -> 22uF
Changed lines of the file:
@@
 Sheet 1 1
 Title "M. Stephan - Mooltipass Schematics (Licensed under CERN OHL V1.2)"
-Date "6 may 2014"
+Date "25 jun 2014"
 Rev "2"
 Comp ""
@@
 P 2450 1550
 F 0 "C1" H 2450 1650 40  0000 L CNN
-F 1 "10uF" H 2456 1465 40  0000 L CNN
+F 1 "22uF" H 2456 1465 40  0000 L CNN
 F 2 "~" H 2488 1400 30  0000 C CNN
 F 3 "~" H 2450 1550 60  0000 C CNN
@@
 P 2700 1550
 F 0 "C3" H 2700 1650 40  0000 L CNN
-F 1 "10uF" H 2706 1465 40  0000 L CNN
+F 1 "22uF" H 2706 1465 40  0000 L CNN
 F 2 "~" H 2738 1400 30  0000 C CNN
 F 3 "~" H 2700 1550 60  0000 C CNN
