File: kicad/olivier_design_v1/mooltipass.kicad_pcb (KiCad board)
At the start: 2 copper layers, 59 parts, among them CON1 AVR-ISP-6, CON2 CON_10118194-0001LF, P1 CONN_8, P2 CONN_6, P3 CONN_10, P4 CONN_8, Q1 MOS_P, Q2 MOS_N, Q3 MOS_P, Q4 MOS_N, U1 CON_SFV30R-2STE1HLF, U2 CON_7312P0225A13LF, U3 IP4234CZ6,125, U4 ATMEGA32U4_QFN, U5 ST662ACD, U6 AT45DB011D-SSH, U7 CON_STACK_9, X1 16MHz

Commit message: working on olivier's design
Parts:
- added R1: 10k, SM0603_Resistor, B.Cu at (118.6, 112.0)
- CON1, Q4: moved to B.Cu
- U3: value IP4234CZ6,125 -> IP4234CZ6,125_ALT
- moved C12 109.8 mm to (116.7, 96.2), turned to 90 degrees
- moved C18 109.6 mm to (124.8, 70.9), turned to 180 degrees
- moved R3 107.8 mm to (138.2, 75.5), turned to 270 degrees
- moved C27 102.4 mm to (132.7, 69.7), turned to 180 degrees
- moved C1 101.8 mm to (138.0, 79.5), turned to 180 degrees
- moved C2 99.6 mm to (141.8, 82.0), turned to 270 degrees
- moved C23 99.4 mm to (129.9, 69.7)
- moved C7 98.7 mm to (114.5, 99.1), turned to 90 degrees
- moved D1 97.2 mm to (135.8, 75.3), turned to 90 degrees
- moved C25 96.9 mm to (132.6, 78.2), turned to 180 degrees
- moved R8 96.2 mm to (119.8, 104.0)
- moved R9 95.9 mm to (119.8, 101.5)
- moved Q3 95.7 mm to (126.5, 73.4), turned to 270 degrees
- moved R5 94.1 mm to (123.8, 73.5), turned to 90 degrees
- moved R10 94.0 mm to (120.8, 97.6), turned to 90 degrees
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Connections:
- net N-0000068 renamed /12V_F
- CON2 pad 2: N-000009 (its old number) -> N-0000010
- CON2 pad 3: N-000003 -> N-000006
- Q4 pad G: (no net) -> /LED_PWM
- U3 pad 1: N-000003 -> N-0000010
- U3 pad 3: /USB_D+ -> /USB_D-
- U3 pad 4: /USB_D- -> /USB_D+
- U3 pad 6: N-000009 (its old number) -> N-000006

Commit message: update schematics olivier
Parts:
- removed CON1: AVR-ISP-6, pin_array_3x2
- added P5: CONN_1, HOLE_FIX_M3_SMALL, F.Cu at (170.1, 84.8)
- added P6: CONN_1, HOLE_FIX_M3_SMALL, F.Cu at (110.1, 71.8)
- added P7: CONN_1, HOLE_FIX_M3_SMALL, F.Cu at (161.1, 133.1)
- added P8: CONN_1, HOLE_FIX_M3_SMALL, F.Cu at (110.1, 129.4)

Commit message: update position connectors
Parts:
- moved CON2 2.50 mm to (112.0, 100.6)
- moved U1 0.90 mm to (150.1, 78.8)
- moved U7 0.73 mm to (113.1, 116.6), turned to 270 degrees
- moved P5 0.06 mm to (170.1, 84.8)
Changed lines of the file:
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@@
-(kicad_pcb (version 3) (host pcbnew "(2013-05-31 BZR 4019)-stable")
+(kicad_pcb (version 3) (host pcbnew "(2013-07-07 BZR 4022)-stable")
   (general
     (links 218)
-    (no_connects 215)
+    (no_connects 218)
     (area 104.355 67.115 173.718333 137.9672)
     (thickness 1.6)
@@
   )
   (module CON_8_THROUGH   locked (layer BOTTOM.Cu)
-    (at 129.8 84.75 180)
+    (at 129.8 84.76 180)
     (fp_text reference P4 (at 0 -4.25 180) (layer Dessous.SilkS)
       (effects (font (size 0.8 0.8) (thickness 0.15)) (justify mirror))
@@
   )
   (module CON_6_THROUGH   locked (layer BOTTOM.Cu)
-    (at 127.25 133.05 180)
+    (at 127.26 133.02 180)
     (fp_text reference P2 (at 0 -4.25 180) (layer Dessous.SilkS)
       (effects (font (size 0.8 0.8) (thickness 0.15)) (justify mirror))
@@
   )
   (module CON_10_THROUGH   locked (layer BOTTOM.Cu)
-    (at 154.2 84.75 180)
+    (at 154.184 84.76 180)
     (fp_text reference P3 (at 0 -4.25 180) (layer Dessous.SilkS)
       (effects (font (size 0.8 0.8) (thickness 0.15)) (justify mirror))
@@
   )
   (module CON_8_THROUGH   locked (layer BOTTOM.Cu)
-    (at 147.6 133.05 180)
+    (at 147.58 133.02 180)
     (fp_text reference P1 (at 0 -4.25 180) (layer Dessous.SilkS)
       (effects (font (size 0.8 0.8) (thickness 0.15)) (justify mirror))
@@
     )
   )
-  (module CON_STACK9_DB9_9S_1V (layer TOP.Cu)
-    (at 113.4 117.25 90)
-    (fp_text reference U7 (at 0 4 90) (layer Dessus.SilkS)
+  (module CON_STACK9_DB9_9S_1V   locked (layer TOP.Cu)
+    (at 113.12 116.58 270)
+    (fp_text reference U7 (at 0 4 270) (layer Dessus.SilkS)
       (effects (font (size 0.8 0.8) (thickness 0.15)))
     )
-    (fp_text value CON_STACK_9 (at 0 0 90) (layer Dessus.SilkS)
+    (fp_text value CON_STACK_9 (at 0 0 270) (layer Dessus.SilkS)
       (effects (font (size 0.8 0.8) (thickness 0.15)))
     )
@@
     (fp_line (start 4.15 2.1) (end -4.15 2.1) (layer Dessus.SilkS) (width 0.15))
     (fp_line (start -4.15 2.1) (end -4.15 -2.1) (layer Dessus.SilkS) (width 0.15))
-    (pad 1 smd rect (at -2 2.1 90) (size 0.7 2.2)
+    (pad 1 smd rect (at -2 2.1 270) (size 0.7 2.2)
       (layers TOP.Cu Dessus.Pate Dessus.Masque)
       (net 3 +5V)
     )
-    (pad 3 smd rect (at -1 2.1 90) (size 0.7 2.2)
+    (pad 3 smd rect (at -1 2.1 270) (size 0.7 2.2)
       (layers TOP.Cu Dessus.Pate Dessus.Masque)
       (net 8 /I2C_SCL)
     )
-    (pad 5 smd rect (at 0 2.1 90) (size 0.7 2.2)
+    (pad 5 smd rect (at 0 2.1 270) (size 0.7 2.2)
       (layers TOP.Cu Dessus.Pate Dessus.Masque)
     )
-    (pad 7 smd rect (at 1 2.1 90) (size 0.7 2.2)
+    (pad 7 smd rect (at 1 2.1 270) (size 0.7 2.2)
       (layers TOP.Cu Dessus.Pate Dessus.Masque)
       (net 13 /LED_CAT)
     )
-    (pad 9 smd rect (at 2 2.1 90) (size 0.7 2.2)
+    (pad 9 smd rect (at 2 2.1 270) (size 0.7 2.2)
       (layers TOP.Cu Dessus.Pate Dessus.Masque)
       (net 46 GND)
     )
-    (pad 4 smd rect (at -0.5 -2.1 90) (size 0.7 2.2)
+    (pad 4 smd rect (at -0.5 -2.1 270) (size 0.7 2.2)
       (layers TOP.Cu Dessus.Pate Dessus.Masque)
       (net 9 /I2C_SDA)
     )
-    (pad 6 smd rect (at 0.5 -2.1 90) (size 0.7 2.2)
+    (pad 6 smd rect (at 0.5 -2.1 270) (size 0.7 2.2)
       (layers TOP.Cu Dessus.Pate Dessus.Masque)
       (net 13 /LED_CAT)
     )
-    (pad 2 smd rect (at -1.5 -2.1 90) (size 0.7 2.2)
+    (pad 2 smd rect (at -1.5 -2.1 270) (size 0.7 2.2)
       (layers TOP.Cu Dessus.Pate Dessus.Masque)
       (net 3 +5V)
     )
-    (pad 8 smd rect (at 1.5 -2.1 90) (size 0.7 2.2)
+    (pad 8 smd rect (at 1.5 -2.1 270) (size 0.7 2.2)
       (layers TOP.Cu Dessus.Pate Dessus.Masque)
       (net 46 GND)
     )
-    (pad FIX1 thru_hole rect (at -3.55 0 90) (size 3.5 4) (drill 2 (offset -0.75 0))
+    (pad FIX1 thru_hole rect (at -3.55 0 270) (size 3.5 4) (drill 2 (offset -0.75 0))
       (layers *.Cu *.Mask Dessus.SilkS)
       (net 46 GND)
     )
-    (pad FIX2 thru_hole rect (at 3.55 0 270) (size 3.5 4) (drill 2 (offset -0.75 0))
+    (pad FIX2 thru_hole rect (at 3.55 0 90) (size 3.5 4) (drill 2 (offset -0.75 0))
       (layers *.Cu *.Mask Dessus.SilkS)
       (net 46 GND)
@@
   )
   (module CON_FPC30   locked (layer BOTTOM.Cu)
-    (at 150.12 77.88)
+    (at 150.12 78.78)
     (fp_text reference U1 (at 0 -3.3) (layer Dessous.SilkS)
       (effects (font (size 1 1) (thickness 0.15)) (justify mirror))
@@
   )
   (module CONUSB_10118194   locked (layer TOP.Cu)
-    (at 111.97 103.08 270)
+    (at 111.97 100.58 270)
     (fp_text reference CON2 (at 0 6.85 270) (layer Dessus.SilkS)
       (effects (font (size 1 1) (thickness 0.15)))
@@
     )
   )
-  (module HOLE_FIX_M3_SMALL (layer TOP.Cu)
-    (at 170.12 84.8422)
+  (module HOLE_FIX_M3_SMALL   locked (layer TOP.Cu)
+    (at 170.12 84.78)
     (fp_text reference P5 (at 0 4.1) (layer Dessus.SilkS)
       (effects (font (size 1 1) (thickness 0.15)))
@@
     )
   )
-  (module HOLE_FIX_M3_SMALL (layer TOP.Cu)
+  (module HOLE_FIX_M3_SMALL   locked (layer TOP.Cu)
     (at 110.12 71.78)
     (fp_text reference P6 (at 0 4.1) (layer Dessus.SilkS)
@@
     )
   )
-  (module HOLE_FIX_M3_SMALL (layer TOP.Cu)
-    (at 161.12 133.1022)
+  (module HOLE_FIX_M3_SMALL   locked (layer TOP.Cu)
+    (at 161.12 133.08)
     (fp_text reference P7 (at 0 4.1) (layer Dessus.SilkS)
       (effects (font (size 1 1) (thickness 0.15)))
@@
     )
   )
-  (module HOLE_FIX_M3_SMALL (layer TOP.Cu)
+  (module HOLE_FIX_M3_SMALL   locked (layer TOP.Cu)
     (at 110.12 129.38)
     (fp_text reference P8 (at 0 4.1) (layer Dessus.SilkS)
