File: kicad/olivier_design_v1/mooltipass.kicad_pcb (KiCad board)
At the start: 4 copper layers, 64 parts, among them CON2 CON_10118194-0001LF, P1 CONN_8, P2 CONN_6, P3 CONN_10, P4 CONN_8, P5 CONN_1, P6 CONN_1, P7 CONN_1, P8 CONN_1, Q1 MOS_P, Q2 MOS_N, Q3 MOS_P, Q4 MOS_N, U1 CON_SFV30R-2STE1HLF, U2 CON_7312P0225A13LF, U3 IP4234CZ6,125, U4 ATMEGA32U4_QFN, U5 ST662ACD, U6 AT45DB011D-SSH, U7 CON_STACK_9, X1 16MHz

Commit message: update Olivier's designs
Parts:
- moved R9 10.4 mm to (126.0, 110.5), turned to 0 degrees
- moved R8 7.71 mm to (125.6, 109.0), turned to 0 degrees
- moved U7 4.47 mm to (111.1, 120.6)
- moved U3 3.69 mm to (117.7, 107.4)
- moved C12 2.75 mm to (111.8, 111.5)
- moved FB1 2.15 mm to (113.5, 108.2)
- moved C7 1.75 mm to (110.5, 107.4)
- moved C15 0.50 mm to (129.4, 111.0)
Routing:
- net +5V: track 111.8 -> 56.1 mm, vias 15 -> 16
- net N-0000059: track 18.3 -> 7.04 mm
- net N-0000060: track 16.0 -> 7.32 mm
- net /USB_D-: track 1.66 -> 9.70 mm
- net /nCHANGE: track 44.1 -> 36.3 mm, vias 1 -> 3
- net GND: track 180.3 -> 186.0 mm, vias 52 -> 51
- net /USB_D+: track 1.66 -> 6.48 mm
- net /LED_CAT: track 8.95 -> 13.4 mm
- net /I2C_SDA: track 157.3 -> 161.0 mm
- net N-0000057: track 6.72 -> 10.2 mm
- net N-0000054: track 8.22 -> 11.6 mm
- net N-0000062: track 17.4 -> 18.9 mm

Commit message: gerbers
Parts:
- moved U3 6.82 mm to (116.0, 100.8), turned to 0 degrees
- moved C11 5.00 mm to (121.8, 102.4)
- moved R1 1.40 mm to (118.6, 113.5)
- moved Q4 1.30 mm to (118.7, 116.2)
- moved R9 0.35 mm to (125.6, 110.5)
Routing:
- net /USB_D+: track 6.48 -> 13.5 mm
- net N-0000057: track 10.2 -> 4.78 mm
- net N-0000054: track 11.6 -> 6.35 mm
- net N-0000062: track 18.9 -> 15.1 mm
- net /USB_D-: track 9.70 -> 12.1 mm
- net /LED_CAT: track 13.4 -> 12.1 mm
- net GND: track 186.0 -> 187.0 mm, vias 51 -> 52

Commit message: final PCBs!
Parts:
- added F1: FUSE, SM1206, B.Cu at (113.7, 94.7)
- U6: footprint SO8E -> SO8EN
- moved C22 4.02 mm to (117.8, 94.9), turned to 0 degrees
- moved U6 0.70 mm to (120.2, 91.2)
- moved R11 0.30 mm to (166.1, 80.2)
Connections:
- C7 pad 1: N-0000062 (its old number) -> VCC
- CON2 pad 1: N-0000062 (its old number) -> N-0000054
- FB1 pad 1: N-0000062 (its old number) -> VCC
- U3 pad 5: N-0000062 (its old number) -> VCC
Routing:
- net VCC: track 0.00 -> 16.6 mm
- net N-0000062 (its old number): track 15.1 -> 0.00 mm, vias 1 -> 0
- net N-0000054: track 0.00 -> 7.81 mm, vias 0 -> 1
- net +3.3V: track 118.1 -> 119.6 mm, vias 5 -> 6
- net /PD2: track 67.4 -> 68.7 mm
- net /SPI2_MOSI: track 48.9 -> 50.0 mm
- net GND: vias 52 -> 53
Other:
- board text added: "Mooltipass M.Stephan / limpkin For Olivier's design Licensed under CERN OHL V1.2"
- board text removed: "Mooltipass with Hackaday M.Stephan / limpkin For Olivier's design"

Commit message: updating bottom PCB
Other:
- board text added: "Mooltipass by M.Stephan Licensed under CERN OHL V1.2"
- board text removed: "Mooltipass M.Stephan / limpkin For Olivier's design Licensed under CERN OHL V1.2"
