File: kicad/olivier_design_v1_top/mooltipass_top.kicad_pcb (KiCad board)
At the start: 2 copper layers, 30 parts, among them K1 CONN_3, P1 CONN_1, P2 CONN_1, P3 CONN_1, P4 CONN_1, U1 CON_STACK_9, U2 AT42QT2120

Commit message: update gerbers
Parts:
- added VAL: solder_top_wheel, solder_top_wheel, F.Cu at (188.2, 148.1)
