File: kicad/mini/kicad_folder/mooltipass_mini.kicad_pcb (KiCad board)
At the start: 2 copper layers, 74.9 x 32.5 mm, 61 parts, among them CON1 CON_10118194-0001LF, Q1 MOS_P, Q2 MOS_N, Q3 MOS_P, Q4 MOS_N, U1 IP4234CZ6,125, U2 ST662ACD, U3 CON_UGM128032A6B01, U4 CON_SMARTCARD2, U5 AT45DB011D, U6 ATMEGA32U4_QFN, U7 LIS2HH12, U8 TS005_WHEEL_CLICK, X1 16MHz

Commit message: updated gerbers and schematics for mini
Parts:
- added P1: EMC, _kicad4_lib:EMC_SMR-TS-3-3-2DGR2E-01, B.Cu at (166.4, 96.8)
- added P2: EMC, _kicad4_lib:EMC_SMR-TS-3-3-2DGR2E-01, B.Cu at (165.9, 72.7)
- added P3: EMC, _kicad4_lib:EMC_SMR-TS-3-3-2DGR2E-01, F.Cu at (168.4, 97.3)
- added P4: EMC, _kicad4_lib:EMC_SMR-TS-3-3-2DGR2E-01, F.Cu at (168.4, 70.2)
- C8: value 1uF -> 100nF
- C9: value 10uF -> 4.7uF; footprint Capacitors_SMD:C_1206 -> Capacitors_SMD:C_0603
- moved C9 0.98 mm to (108.7, 88.7)
Routing:
- net GND: track 195.6 -> 199.2 mm, vias 55 -> 58
- net /SPI_SCK: track 47.3 -> 48.1 mm
Other:
- board text added: "Mooltipass Mini by Stephan Electronics Licensed under CERN OHL V1.2 v4"
- board text removed: "Mooltipass Mini by Stephan Electronics Licensed under CERN OHL V1.2 v3"
