File: kicad/mini/kicad_folder/mooltipass_mini.sch (KiCad schematic (older format))
At the start: 61 parts, among them CON1 CON_10118194-0001LF, Q1 MOS_P, Q2 MOS_N, Q3 MOS_P, Q4 MOS_N, U1 IP4234CZ6,125, U2 ST662ACD, U3 CON_UGM128032A6B01, U4 CON_SMARTCARD2, U5 AT45DB011D, U6 ATMEGA32U4_QFN, U7 LIS2HH12, U8 TS005_WHEEL_CLICK, X1 16MHz

Commit message: updated gerbers and schematics for mini
Parts:
- added P1, P2, P3, P4: EMC, _kicad4_lib:EMC_SMR-TS-3-3-2DGR2E-01, symbol CONN_01X01
- C8: value 1uF -> 100nF
- C9: value 10uF -> 4.7uF; footprint Capacitors_SMD:C_1206 -> Capacitors_SMD:C_0603
Connections:
- net GND: now also P1.1 (P1), P2.1 (P1), P3.1 (P1), P4.1 (P1)
Other:
- note added: "|041E/081E/161E/321E"
- moved on the sheet: C9
