File: kicad/mini/kicad_folder_smc_chinese_con/mooltipass_mini.sch (KiCad schematic (older format))
At the start: 65 parts, among them CON1 CON_10118194-0001LF, P1 EMC, P2 EMC, P3 EMC, P4 EMC, Q1 MOS_P, Q2 MOS_N, Q3 MOS_P, Q4 MOS_N, U1 IP4234CZ6,125, U2 ST662ACD, U3 CON_UGM128032A6B01, U4 CON_SMARTCARD2, U5 AT45DB011D, U6 ATMEGA32U4_QFN, U7 LIS2HH12, U8 TS005_WHEEL_CLICK, X1 16MHz

Commit message: final gerbers for mini with chinese card connector clone
Parts:
- C9: footprint Capacitors_SMD:C_1206 -> Capacitors_SMD:C_0603
- U4: footprint _kicad4_lib:CON_SMARTCARD_5145300-3 -> _kicad4_lib:CON_SMARTCARD_CLONE_91-90473-003A
Changed lines of the file:
@@
 F 0 "C9" H 6560 1570 50  0000 L CNN
 F 1 "4.7uF" H 6560 1420 50  0000 L CNN
-F 2 "Capacitors_SMD:C_1206" H 6550 1500 50  0001 C CNN
+F 2 "Capacitors_SMD:C_0603" H 6550 1500 50  0001 C CNN
 F 3 "" H 6550 1500 50  0000 C CNN
 	1    6550 1500
@@
 F 0 "U4" H 4250 3350 60  0000 C CNN
 F 1 "CON_SMARTCARD2" H 4500 2250 60  0000 C CNN
-F 2 "_kicad4_lib:CON_SMARTCARD_5145300-3" H 3700 3400 60  0001 C CNN
+F 2 "_kicad4_lib:CON_SMARTCARD_CLONE_91-90473-003A" H 3700 3400 60  0001 C CNN
 F 3 "" H 3700 3400 60  0000 C CNN
 	1    4500 2800
